File: Other_Files/Controllers/PCBs/Controller_Bluetooth/Right_Controller_PCB_Bluetooth/Right_Controller_PCB_Bluetooth.kicad_sch (KiCad schematic)
At the start: 13 parts

Commit message: Updated the Controllers' PCB to version 1.2
Parts:
- H1, H2, H3, H4: footprint MountingHole:MountingHole_3mm -> MountingHole:MountingHole_3.2mm_M3
Changed lines of the file:
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@@
 			)
 		)
-		(property "Footprint" "MountingHole:MountingHole_3mm"
+		(property "Footprint" "MountingHole:MountingHole_3.2mm_M3"
 			(at 101.6 190.5 0)
 			(effects
@@
 			)
 		)
-		(property "Footprint" "MountingHole:MountingHole_3mm"
+		(property "Footprint" "MountingHole:MountingHole_3.2mm_M3"
 			(at 25.4 190.5 0)
 			(effects
@@
 			)
 		)
-		(property "Footprint" "MountingHole:MountingHole_3mm"
+		(property "Footprint" "MountingHole:MountingHole_3.2mm_M3"
 			(at 50.8 190.5 0)
 			(effects
@@
 			)
 		)
-		(property "Footprint" "MountingHole:MountingHole_3mm"
+		(property "Footprint" "MountingHole:MountingHole_3.2mm_M3"
 			(at 76.2 190.5 0)
 			(effects

Commit message: Updated Bluetooth Controllers' PCBs
Connections:
- net A: now also CentralBoard1.8 (D5); no longer CentralBoard1.7 (D4)
- net B: now also CentralBoard1.9 (D6); no longer CentralBoard1.6 (D3)
- net SEL_JOY_R: now also CentralBoard1.15 (D12); no longer CentralBoard1.9 (D6)
- net START_R: now also CentralBoard1.5 (D2); no longer CentralBoard1.10 (D7)
- net X: now also CentralBoard1.7 (D4); no longer CentralBoard1.8 (D5)
- net Y: now also CentralBoard1.6 (D3); no longer CentralBoard1.5 (D2)
